Commit message: panda urdf updated

File: franka_panda_mod/panda.urdf (robot description, URDF)
Before this commit: robot panda, 9 links, 8 joints
Links:
- added link paddle_2_v11, mass 0.41109102084948795; collision mesh filename=package://meshes/collision/paddle_2_v11.stl scale=0.001 0.001 0.001; visual mesh filename=package://meshes/collision/paddle_2_v11.stl scale=0.001 0.001 0.001
Joints:
- added joint panda_bat_mount: type fixed, parent panda_link8, child paddle_2_v11, origin xyz=0.0 0.0 0.0 rpy=3.4416 0 0
