Commit message: pingpong paddle added to panda

File: modURDFs/panda_pybullet/franka_panda_mod/panda.urdf (robot description, URDF)
Before this commit: robot panda, 11 links, 10 joints
Links:
- link end_effector_1: geometry collision mesh filename=package://meshes/visual/end_effector1.stl scale=0.001 0.001 0.001; visual mesh filename=package://meshes/visual/end_effector1.stl scale=0.001 0.001 0.001
- link racquet_1: geometry collision mesh filename=package://meshes/visual/paddle_2_v11.stl scale=0.001 0.001 0.001; visual mesh filename=package://meshes/visual/paddle_2_v11.stl scale=0.001 0.001 0.001

Commit message: In Sha Allah

File: modURDFs/panda_pybullet/franka_panda_mod/panda.urdf (robot description, URDF)
Before this commit: robot panda, 11 links, 10 joints
Links:
- removed link end_effector_1
- removed link racquet_1
- added link paddle_2_v11, mass 0.41109102084948795; collision mesh filename=package://meshes/collision/paddle_2_v11.stl scale=0.001 0.001 0.001; visual mesh filename=package://meshes/collision/paddle_2_v11.stl scale=0.001 0.001 0.001
Joints:
- removed joint panda_racquet_mount
- removed joint racquet_endeff
- added joint panda_bat_mount: type fixed, parent panda_link8, child paddle_2_v11, origin xyz=0.0 0.0 0.0 rpy=3.4416 0 0

Commit message: urdf updated

File: modURDFs/panda_pybullet/franka_panda_mod/panda.urdf (robot description, URDF)
Before this commit: robot panda, 10 links, 9 joints
Links:
- added link end_eff1, mass 0.003088967880428063; collision mesh filename=package://meshes/collision/end_eff1.stl scale=0.001 0.001 0.001; visual mesh filename=package://meshes/collision/end_eff1.stl scale=0.001 0.001 0.001
Joints:
- added joint Rigid_27: type fixed, parent paddle_2_v11, child end_eff1, origin xyz=0.001106 -0.041099 -0.175399 rpy=0 0 0
